File: NU-Smarticle PCB Design/Eagle Files/NU-Smarticles/NU-Smarticles.sch (EAGLE design)
At the start: 66 parts, among them IC1 CP2104, IC2 ATMEGA328P, Q3 DMG341, SW2 KMR2, U6 AP2112-3.3, U7 MCP73831T-2ACI/OT, U8 OPA344, U9 ADMP401, X1 JSTPH, X4 20329, Y2 CSTCE16M0V53-R0 8MHZ

Commit message: include v2 Smarticles
Parts:
- removed C20, C21: 10uF, microbuilder:CAP_CERAMIC0805-NOOUTLINE
- removed C22, C23, C24, C25: 0.1uF, microbuilder:CAP_CERAMIC0603_NO
- removed C26: 10uF, microbuilder:CAP_CERAMIC_0805MP
- removed C27, C28: 1uF, microbuilder:CAP_CERAMIC0603_NO
- removed C29: 100pF, SparkFun-Capacitors:100PF-0603-50V-5%
- removed C30: 4.7uF, SparkFun-Capacitors:4.7UF0603
- removed C31: 1.0uF, SparkFun-Capacitors:1.0UF-0603-16V-10%
- removed C32: 0.1uF, SparkFun-Capacitors:0.1UF-0603-25V-5%
- removed D6: RED, microbuilder:LED0805_NOOUTLINE
- removed D7, D8: YELLOW, microbuilder:LED0805_NOOUTLINE
- removed FRAME1: FRAME-LETTER, SparkFun-Aesthetics:FRAME-LETTER
- removed PR4, PR5, PR6: A1050_09, photo-elements:A1050_09
- removed R10, R11, R12, R15, R24: 10k, SparkFun-Resistors:10KOHM-0603-1/10W-1%
- removed R16, R17, R22, R23: 1K, microbuilder:RESISTOR_0603_NOOUT
- removed R18, R19: 10K, microbuilder:RESISTOR_0603_NOOUT
- removed R20: 100K, microbuilder:RESISTOR_4PACK
- removed R21: 1K, microbuilder:RESISTOR_0603MP
- removed R25: 1.5k, SparkFun-Resistors:1.5KOHM-0603-1/10W-1%
- removed R26: 100k, SparkFun-Resistors:100KOHM-0603-1/10W-1%
- removed SW2: KMR2, microbuilder:SWITCH_TACT_SMT4.6X2.8
- removed U$31, U$32: MOUNTINGHOLE2.5, microbuilder:MOUNTINGHOLE2.5
- removed U$34, U$35: FIDUCIAL_1MM, microbuilder:FIDUCIAL_1MM
- removed X4: 20329, microbuilder:USB_MICRO_20329_V2
- added C10, C4, C5, C9: 0.1uF, NU-Smarticles:CAP_CERAMIC_0402MP
- added C11, C8: 1uF, NU-Smarticles:CAP_CERAMIC_0402MP
- added C12: 9.0pF, NU-Smarticles:CAP_CERAMIC_0402MP
- added C13: 1.0uF, NU-Smarticles:CAP_CERAMIC_0402MP
- added C14: 4.7uF, NU-Smarticles:CAP_CERAMIC_0402MP
- added C2, C7: 10uF, NU-Smarticles:CAP_CERAMIC_0402MP
- added C3: 10µF, microbuilder:CAP_CERAMIC_0402MP
- added C6: 10µF, NU-Smarticles:CAP_CERAMIC_0402MP
- added PH1, PH2, PH3: A1050_09, NU-Smarticles:A1050_09
- added Q1: DMG341, microbuilder:MOSFET-P
- added R1: 1.5k, NU-Smarticles:RESISTOR_0402MP
- added R101: 1K, microbuilder:RESISTOR_0402MP
- added R102: 1k, NU-Smarticles:RESISTOR_0402MP
- added R104: 10K, microbuilder:RESISTOR_0402MP
- added R108, R3, R4, R6, R7, R8: 10k, NU-Smarticles:RESISTOR_0402MP
- added R5, R9: 100k, NU-Smarticles:RESISTOR_0402MP
- added S1: (no value), NU-Smarticles:SWITCH-SPDT-SMD-AYZ0202
- added U$56: LI-PO, NU-Smarticles:LI-PO
- C1: value 0.1uF -> 10uF; device SparkFun-Capacitors:0.1UF-0603-25V-5% -> NU-Smarticles:CAP_CERAMIC_0402MP
- C15: value 9.0pF -> 1.0uF; device SparkFun-Capacitors:9.0PF-0603-50V-10% -> NU-Smarticles:CAP_CERAMIC_0402MP
- C16: value 1.0uF -> 100pF; device SparkFun-Capacitors:1.0UF-0603-16V-10% -> NU-Smarticles:CAP_CERAMIC_0402MP
- C17, C18: value 10µF -> 0.1uF; device microbuilder:CAP_CERAMIC0805-NOOUTLINE -> NU-Smarticles:CAP_CERAMIC_0402MP
- CHG: device microbuilder:LED0805_NOOUTLINE -> microbuilder:LED0603
- D5: device microbuilder:DIODE-SCHOTTKYSOD-123 -> microbuilder:DIODE-SCHOTTKYSOD-523
- IC1: value CP2104 -> CP2102N
- R2: device SparkFun-Resistors:0.1OHM-1210-1/2W-1% -> NU-Smarticles:RESISTOR_0603MP
- U6: device microbuilder:VREG_SOT23-5 -> NU-Smarticles:VREG_SOT23-5
- X1: value JSTPH -> (none); device microbuilder:CON_JST_PH_2PIN -> Adafruit Feather 328P:USBMICRO_20329
Connections:
- removed net N$21: IC1G$1.D+, X4.D+
- removed net N$22: IC1G$1.D-, X4.D-
- removed net N$24: D6.A, R17.2
- removed net N$25: D7.A, R23.1
- removed net N$26: D8.A, R22.1
- removed net RXLED1: D7.C, IC1G$1.GPIO1/RXLED
- removed net TXLED1: D8.C, IC1G$1.GPIO0/TXLED
- removed net VBAT: C18.1, JP5.1, Q3.D, R20G$2.1, U7.VBAT, X1.2
- removed net VBUS: C27.2, CHG.A, D5.A, IC1G$1.REGIN, IC1G$1.VBUS, JP5.3, Q3.G, R20G$4.1, R22.2, R23.2, U7.VDD, X4.VBUS
- new net N$2: IC1G$1.D+, X1.D+
- new net N$3: IC1G$1.D-, X1.D-
- new net VCC_1: JP5.1, Q1.D, R2.1, U$47.IN+
- new net VIN: S1.P, U$56.+
- new net V_USB: C8.2, CHG.A, D5.A, IC1G$1.REGIN, IC1G$1.VBUS, JP5.3, Q1.G, Q3.G, R9.2, U7.VDD, X1.VBUS
- new net XB_DTR: J1.1, U$2.DTR
- new net XB_RTS: J1.2, U$2.RTS
- net 3.3V: now also C10.2, C12.2, C13.2, C17.1, C18.1, C2.1, C9.2, J1.5, JP4.4, PH1.1, PH2.1, PH3.1, R108.2, R3.2; no longer C15.2, C16.2, C20.1, C21.1, C24.2, C25.2, C32.1, PR4.1, PR5.1, PR6.1, R15.2, R19.2
- net A0: now also PH1.2, R6.2; no longer PR6.2, R12.2
- net A1: now also PH2.2, R7.2; no longer PR4.2, R10.2
- net A2: now also PH3.2, R8.2; no longer PR5.2, R11.2
- net A3: now also C16.2, R5.2; no longer C29.2, R26.1
- net A5: no longer JP5.11
- net A6: no longer JP4.8, R20G$2.2, R20G$3.2
- net A7: no longer JP4.7
- net AREF: now also C4.2; no longer C22.2, JP4.14
- net D0/RX: now also R101.1; no longer R21.1
- net D10: now also J1.4, U$2.DIN
- net D11: no longer JP4.5
- net D12: no longer JP4.4
- net D13: no longer JP4.6, R17.1
- net D2: no longer JP5.6
- net D5: no longer JP5.10
- net D6: no longer JP5.9
- net D7: no longer JP4.1
- net D8: no longer U$2.DIN
- net D9: now also J1.3
- net DTR: now also C5.1; no longer C23.1
- net GND: now also C10.1, C11.2, C12.1, C13.1, C15.2, C2.2, C3.2, C4.1, C6.2, C7.2, C8.1, C9.1, J1.6, JP4.6, R104.1, R4.1, R6.1, R7.1, R8.1, R9.1, U$56.-, X1.GND; no longer C15.1, C16.1, C20.2, C21.2, C22.1, C24.1, C25.1, C26.2, C27.1, C28.2, C31.2, C32.2, D6.C, R10.1, R11.1, R12.1, R18.1, R20G$3.1, R20G$4.2, R24.1, SW2.P, SW2.P1, X1.1, X4.GND
- net N$16: now also C14.1; no longer C30.1
- net N$17: now also C16.1, R1.2, R5.1; no longer C29.1, R25.1, R26.2
- net N$18: now also R102.1; no longer R16.1
- net N$19: now also R102.2; no longer R16.2
- net N$20: now also R104.2; no longer R18.2
- net N$23: now also C6.1; no longer C17.1
- net N$27: now also C11.1; no longer C28.1
- net N$29: now also C14.2, R1.1; no longer C30.2, R25.2
- net N$30: now also C15.1, R3.1, R4.2; no longer C31.1, R15.1, R24.2
- net N$41: now also C7.1; no longer C26.1
- net RESET: now also C5.2, JP4.1, R108.1; no longer C23.2, R19.1, SW2.S, SW2.S1
- net RXD: now also R101.2; no longer R21.2
- net V_BATT: now also C3.1, Q1.S, Q3.D, S1.O, U7.VBAT; no longer R2.1, U$47.IN+
Other:
- note removed: "Assorted"
- note removed: "RESET"
