Commit message: new urdf

File: simulation_urdf/urdf/simulation_urdf.urdf (robot description, URDF)
Before this commit: robot Smarticle_URDF, 3 links, 2 joints
Links:
- link base_link: mass 0.0269834813442291 -> 0.0461924870615736; geometry collision mesh filename=package://simulation_urdf/meshes/base_link.STL; visual mesh filename=package://simulation_urdf/meshes/base_link.STL
- link left_arm: mass 0.00390817547516661 -> 0.00328492067362327; geometry collision mesh filename=package://simulation_urdf/meshes/left_arm.STL; visual mesh filename=package://simulation_urdf/meshes/left_arm.STL
- link right_arm: mass 0.00390817547516661 -> 0.00328492067362327; geometry collision mesh filename=package://simulation_urdf/meshes/right_arm.STL; visual mesh filename=package://simulation_urdf/meshes/right_arm.STL
Joints:
- removed joint left_servo
- removed joint right_servo
- added joint left_joint: type continuous, parent base_link, child left_arm, origin xyz=0.0482 0.0135 0 rpy=1.5708 0 3.0427, axis 0 1 0, limit lower=-3.15 upper=3.15 effort=0.04 velocity=6.28
- added joint right_joint: type continuous, parent base_link, child right_arm, origin xyz=0.0058 0.0135 0 rpy=1.5708 0 0, axis 0 1 0, limit lower=-3.15 upper=3.15 effort=0.04 velocity=6.28
