File: NU-Smarticle PCB Design/Eagle Files/NU-Smarticles-v2.0/topboard-v2.0.brd (EAGLE design)
At the start: 48 x 22 mm, 17 parts, among them CON1 LI-PO, CON2 12XFFCEXTEND, M1 SERVO, M2 SERVO, U1 XBEE3, U2 INA180B2

Commit message: eagle work and files added
Parts:
- removed CON2: 12XFFCEXTEND, NU-Smarticle v2:15166-0117_XTEND
- removed R4: 10k, NU-Smarticle v2:_0603MP
- removed U2: INA180B2, NU-Smarticle v2:SOT23-5
- added CON100: 12XFFCMOLEX_51281, NU-Smarticle v2:MOLEX_51281-1294
- added R100: 0.1, NU-Smarticle v2:_0603MP
- added U100: INA180B2, NU-Smarticle v2:SOT23-5
- C1: value 0.1uF -> 9.0pF
- C2: value 9.0pF -> 1.0uF
- C3: value 1.0uF -> 0.1uF
- R1: value 0.1 -> 10k
- moved PH2 45.6 mm to (45.3, 4.19), turned to 270 degrees
- moved PH1 37.1 mm to (11.6, 17.4), turned to 180 degrees
- moved R3 36.9 mm to (41.7, 1.72), turned to 270 degrees
- moved R2 30.0 mm to (11.9, 2.46), turned to 90 degrees
- moved M1 28.8 mm to (9.75, 4.23), turned to 180 degrees
- moved M2 28.8 mm to (38.4, 4.18), turned to 0 degrees
- moved R1 16.2 mm to (14.2, 11.5), flipped to the top, turned to 90 degrees
- moved C1 12.3 mm to (15.3, 16.2), turned to 270 degrees
- moved C3 5.27 mm to (14.3, 7.99), turned to 0 degrees
- moved PH3 5.04 mm to (5.72, 2.44), turned to 0 degrees
- moved C2 3.12 mm to (14.1, 16.2)
- moved CON1 3.00 mm to (33.9, 2.17)
- moved S1 3.00 mm to (43.3, 20.0)
- moved U1 3.00 mm to (24.2, 11.9)
Connections:
- removed net D2: CON2.P7, U1.DOUT/DIO13
- removed net D3: CON2.P8, U1.DIN/CONFIG/DIO14
- removed net D4: CON2.P9, M1.1
- new net D9: CON100.P11, M1.1
- new net RXD1: CON100.P3, U1.DOUT/DIO13
- new net TXD1: CON100.P4, U1.DIN/CONFIG/DIO14
- net 3.3V: now also C1.2, CON100.P1, U100.5; no longer C1.1, CON2.P10, U2.2
- net A0: now also CON100.P6, PH2.2, R3.2; no longer CON2.P5, PH1.2, R2.2
- net A1: now also CON100.P7, U100.4; no longer CON2.P4, U2.4
- net A2: now also CON100.P8, PH3.2, R2.2; no longer CON2.P3, PH2.2, R3.2
- net A3: now also CON100.P9, PH1.2, R1.2; no longer CON2.P2, PH3.2, R4.2
- net D10: now also CON100.P2; no longer CON2.P0
- net GND: now also C1.1, CON100.P5, R1.1, U100.2; no longer C1.2, CON2.P6, R4.1, U2.5
- net N$1: now also R100.2, U100.3; no longer R1.2, U2.3
- net VBAT: now also CON100.P0; no longer CON2.P11
- net VCC_1: now also R100.1, U100.1; no longer R1.1, U2.1
Routing:
- net D4: track 25.5 -> 0.00 mm, vias 2 -> 0
- net D3: track 16.5 -> 0.00 mm, vias 1 -> 0
- net D2: track 14.1 -> 0.00 mm, vias 1 -> 0
- net D9: track 0.00 -> 13.3 mm, vias 0 -> 1
- net RXD1: track 0.00 -> 12.4 mm, vias 0 -> 1
- net GND: track 12.4 -> 24.3 mm, vias 2 -> 5
- net TXD1: track 0.00 -> 11.2 mm, vias 0 -> 1
- net A0: track 34.9 -> 25.2 mm, vias 3 -> 1
- net A2: track 27.5 -> 18.7 mm
- net A3: track 28.1 -> 35.5 mm, vias 1 -> 3
- net A1: track 6.95 -> 2.53 mm
- net D10: track 18.3 -> 14.4 mm
- net 3.3V: track 16.6 -> 13.4 mm, vias 2 -> 1
- net VCC_1: track 35.3 -> 33.2 mm
- net VBAT: track 31.9 -> 30.6 mm
Other:
- outline, holes or cut-outs redrawn

Commit message: delete cam outputs
Parts:
- moved PH3 4.00 mm to (9.72, 2.44)
- moved M1 2.00 mm to (9.75, 6.23)
- moved R2 2.00 mm to (13.9, 2.46)
- moved M2 1.00 mm to (38.4, 5.18)
Connections:
- net N$1 renamed IN-
- new net IN+: R100.1, U100.1
- net VCC_1: no longer R100.1, U100.1
Routing:
- net IN-: track 71.8 -> 43.2 mm
- net VCC_1: track 33.2 -> 22.3 mm
- net A2: track 18.7 -> 14.9 mm
- net IN+: track 0.00 -> 1.40 mm
- net 3.3V: track 13.4 -> 14.6 mm
Changed lines of the file:
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@@
 <setting verticaltext="up"/>
 </settings>
-<grid distance="1" unitdist="mm" unit="mm" style="lines" multiple="1" display="no" altdistance="0.01" altunitdist="mm" altunit="mm"/>
+<grid distance="50" unitdist="mil" unit="mil" style="lines" multiple="1" display="no" altdistance="5" altunitdist="mil" altunit="mil"/>
 <layers>
 <layer number="1" name="Top" color="4" fill="1" visible="yes" active="yes"/>
@@
 <layer number="28" name="bValues" color="7" fill="1" visible="no" active="yes"/>
 <layer number="29" name="tStop" color="7" fill="3" visible="no" active="yes"/>
-<layer number="30" name="bStop" color="7" fill="6" visible="no" active="yes"/>
+<layer number="30" name="bStop" color="7" fill="6" visible="yes" active="yes"/>
 <layer number="31" name="tCream" color="7" fill="4" visible="no" active="yes"/>
 <layer number="32" name="bCream" color="7" fill="5" visible="no" active="yes"/>
@@
 <elements>
 <element name="U1" library="NU-Smarticle v2" package="XBEE3_MICRO" value="XBEE3" x="24.19" y="11.94405" smashed="yes"/>
-<element name="M2" library="NU-Smarticle v2" package="1X03_SERVO" value="SERVO" x="38.37" y="4.184" smashed="yes"/>
-<element name="M1" library="NU-Smarticle v2" package="1X03_SERVO" value="SERVO" x="9.75" y="4.229" smashed="yes" rot="R180"/>
+<element name="M2" library="NU-Smarticle v2" package="1X03_SERVO" value="SERVO" x="38.37" y="5.184" smashed="yes"/>
+<element name="M1" library="NU-Smarticle v2" package="1X03_SERVO" value="SERVO" x="9.75" y="6.229" smashed="yes" rot="R180"/>
 <element name="R3" library="NU-Smarticle v2" package="_0603MP" value="10k" x="41.711" y="1.721" smashed="yes" rot="R270">
 <attribute name="NAME" x="39.8235" y="1.15" size="0.6096" layer="25" ratio="18"/>
@@
 <attribute name="NAME" x="13.96" y="13.1865" size="0.6096" layer="25" ratio="18" rot="R90"/>
 </element>
-<element name="R2" library="NU-Smarticle v2" package="_0603MP" value="10k" x="11.914" y="2.457" smashed="yes" rot="R90">
-<attribute name="NAME" x="13.751" y="2.1187" size="0.6096" layer="25" ratio="18" rot="R180"/>
+<element name="R2" library="NU-Smarticle v2" package="_0603MP" value="10k" x="13.914" y="2.457" smashed="yes" rot="R90">
+<attribute name="NAME" x="15.751" y="2.1187" size="0.6096" layer="25" ratio="18" rot="R180"/>
 </element>
 <element name="C2" library="NU-Smarticle v2" package="_0603MP" value="1.0uF" x="14.056" y="16.204" smashed="yes" rot="R270">
@@
 <element name="PH2" library="NU-Smarticle v2" package="PHOTORESISTOR" value="A10" x="45.291" y="4.191" smashed="yes" rot="R270"/>
 <element name="PH1" library="NU-Smarticle v2" package="PHOTORESISTOR" value="A10" x="11.557" y="17.447" smashed="yes" rot="R180"/>
-<element name="PH3" library="NU-Smarticle v2" package="PHOTORESISTOR" value="A10" x="5.7178" y="2.4384" smashed="yes"/>
+<element name="PH3" library="NU-Smarticle v2" package="PHOTORESISTOR" value="A10" x="9.7178" y="2.4384" smashed="yes"/>
 <element name="S1" library="CabelBot" package="SWITCH_SPST_SMD_A" package3d_urn="urn:adsk.eagle:package:40179/1" value="" x="43.307" y="20.018" smashed="yes">
 <attribute name="PROD_ID" value="SWCH-10651" x="43.307" y="20.018" size="1.778" layer="27" display="off"/>
@@
 <wire x1="15.24" y1="14.303" x2="15.24" y2="8.143" width="0.254" layer="1"/>
 <wire x1="15.24" y1="8.143" x2="15.083" y2="7.986" width="0.254" layer="1"/>
-<wire x1="26.65" y1="7.7" x2="26.65" y2="8.87" width="0.254" layer="16"/>
-<wire x1="26.65" y1="7.7" x2="26.67" y2="7.68" width="0.254" layer="16"/>
-<wire x1="26.67" y1="7.68" x2="26.67" y2="6.858" width="0.254" layer="16"/>
+<wire x1="26.65" y1="7.7" x2="26.65" y2="8.87" width="0.2032" layer="16"/>
+<wire x1="26.65" y1="8.87" x2="26.67" y2="8.89" width="0.2032" layer="16"/>
+<wire x1="26.6702" y1="7.17375" x2="26.84875" y2="6.9952" width="0.2032" layer="16"/>
+<wire x1="26.67" y1="8.89" x2="26.6702" y2="8.8898" width="0.2032" layer="16"/>
+<wire x1="26.6702" y1="8.8898" x2="26.6702" y2="7.17375" width="0.2032" layer="16"/>
 </signal>
 <signal name="GND">
@@
 <contactref element="PH3" pad="2"/>
 <contactref element="R2" pad="2"/>
-<wire x1="7.6228" y1="2.4384" x2="8.4034" y2="3.219" width="0.254" layer="1"/>
-<wire x1="8.4034" y1="3.219" x2="11.914" y2="3.219" width="0.254" layer="1"/>
+<wire x1="11.6228" y1="2.4384" x2="12.4034" y2="3.219" width="0.254" layer="1"/>
+<wire x1="12.4034" y1="3.219" x2="13.914" y2="3.219" width="0.254" layer="1"/>
 <via x="15.367" y="4.191" extent="1-16" drill="0.508"/>
-<wire x1="11.914" y1="3.219" x2="12.4668" y2="3.7718" width="0.254" layer="1"/>
-<wire x1="12.4668" y1="3.7718" x2="14.19738125" y2="3.7718" width="0.254" layer="1"/>
+<wire x1="13.914" y1="3.219" x2="13.914" y2="3.48841875" width="0.254" layer="1"/>
+<wire x1="14.61658125" y1="4.191" x2="13.914" y2="3.48841875" width="0.254" layer="1"/>
 <wire x1="14.61658125" y1="4.191" x2="15.367" y2="4.191" width="0.254" layer="1"/>
-<wire x1="14.19738125" y1="3.7718" x2="14.61658125" y2="4.191" width="0.254" layer="1"/>
 <wire x1="23.15" y1="7.148" x2="23.15" y2="7.7" width="0.254" layer="16"/>
 <wire x1="16.2052" y1="5.2408" x2="16.2052" y2="5.77961875" width="0.254" layer="16"/>
@@
 <wire x1="26.2636" y1="7.08035" x2="26.2636" y2="6.35" width="0.2032" layer="16"/>
 <wire x1="26.2636" y1="6.35" x2="26.7716" y2="5.842" width="0.3048" layer="16"/>
-<wire x1="36.712" y1="5.842" x2="38.37" y2="4.184" width="0.3048" layer="16"/>
-<wire x1="26.7716" y1="5.842" x2="36.712" y2="5.842" width="0.3048" layer="16"/>
+<wire x1="37.712" y1="5.842" x2="38.37" y2="5.184" width="0.3048" layer="16"/>
+<wire x1="26.7716" y1="5.842" x2="37.712" y2="5.842" width="0.3048" layer="16"/>
 </signal>
 <signal name="VCC_1">
-<contactref element="U100" pad="1"/>
-<contactref element="R100" pad="1"/>
-<wire x1="24.641" y1="1.524" x2="24.956" y2="2.093" width="0.508" layer="16"/>
-<wire x1="24.956" y1="2.093" x2="24.956" y2="2.8429" width="0.508" layer="16"/>
 <contactref element="S1" pad="2"/>
 <wire x1="42.557" y1="18.268" x2="41.9912" y2="17.5752" width="0.508" layer="1"/>
@@
 <wire x1="41.63258125" y1="16.97" x2="35.052" y2="16.97" width="0.508" layer="1"/>
 <via x="33.782" y="4.5212" extent="1-16" drill="0.508"/>
-<wire x1="24.956" y1="2.8429" x2="26.6371" y2="4.524" width="0.508" layer="16"/>
-<wire x1="26.6371" y1="4.524" x2="33.782" y2="4.5212" width="0.508" layer="16"/>
 <wire x1="32.512" y1="14.43" x2="35.052" y2="16.97" width="0.508" layer="1"/>
 <wire x1="33.782" y1="4.5212" x2="32.512" y2="5.794" width="0.508" layer="1"/>
@@
 <wire x1="27.15" y1="7.7" x2="27.1552" y2="7.7" width="0.254" layer="16"/>
 </signal>
-<signal name="N$1">
+<signal name="IN-">
 <contactref element="U100" pad="3"/>
 <contactref element="R100" pad="2"/>
@@
 <wire x1="23.056" y1="2.8429" x2="23.056" y2="1.839" width="0.508" layer="16"/>
 <wire x1="23.056" y1="1.839" x2="23.117" y2="1.524" width="0.508" layer="16"/>
-<wire x1="46.482" y1="0.5842" x2="24.13" y2="0.5842" width="0.508" layer="16"/>
-<wire x1="24.13" y1="0.5842" x2="23.371" y2="1.3432" width="0.508" layer="16"/>
+<wire x1="23.8571" y1="0.8571" x2="23.371" y2="1.3432" width="0.508" layer="16"/>
 <wire x1="23.371" y1="1.3432" x2="23.117" y2="1.524" width="0.508" layer="16"/>
 <wire x1="23.117" y1="1.524" x2="22.434" y2="0.587" width="0.508" layer="16"/>
-<wire x1="1.27" y1="0.587" x2="0.5842" y2="1.2728" width="0.508" layer="16"/>
-<wire x1="0.5842" y1="4.4732" x2="1.5268" y2="5.4158" width="0.508" layer="16"/>
-<wire x1="22.434" y1="0.587" x2="1.27" y2="0.587" width="0.508" layer="16"/>
-<wire x1="0.5842" y1="1.2728" x2="0.5842" y2="4.4732" width="0.508" layer="16"/>
-<wire x1="46.482" y1="5.4158" x2="47.4158" y2="4.482" width="0.508" layer="16"/>
-<wire x1="47.4158" y1="1.518" x2="46.482" y2="0.5842" width="0.508" layer="16"/>
-<wire x1="47.4158" y1="4.482" x2="47.4158" y2="1.518" width="0.508" layer="16"/>
-<wire x1="6.5312" y1="5.4158" x2="7.718" y2="4.229" width="0.508" layer="16"/>
-<wire x1="1.5268" y1="5.4158" x2="6.5312" y2="5.4158" width="0.508" layer="16"/>
-<wire x1="40.402" y1="4.184" x2="41.6338" y2="5.4158" width="0.508" layer="16"/>
-<wire x1="41.6338" y1="5.4158" x2="46.482" y2="5.4158" width="0.508" layer="16"/>
+<wire x1="22.434" y1="0.587" x2="9" y2="0.587" width="0.508" layer="16"/>
+<wire x1="9" y1="0.587" x2="7.718" y2="1.869" width="0.508" layer="16"/>
+<wire x1="7.718" y1="1.869" x2="7.718" y2="6.229" width="0.508" layer="16"/>
+<wire x1="23.8571" y1="0.8571" x2="23.86131875" y2="0.8571" width="0.508" layer="16"/>
+<wire x1="23.86131875" y1="0.8571" x2="24.05161875" y2="0.6668" width="0.508" layer="16"/>
+<wire x1="24.05161875" y1="0.6668" x2="38.6668" y2="0.6668" width="0.508" layer="16"/>
+<wire x1="40.402" y1="2.402" x2="40.402" y2="5.184" width="0.508" layer="16"/>
+<wire x1="38.6668" y1="0.6668" x2="40.402" y2="2.402" width="0.508" layer="16"/>
 </signal>
 <signal name="RXD1">
@@
 <wire x1="17.479" y1="7.7" x2="15.367" y2="5.588" width="0.254" layer="16"/>
 <via x="15.367" y="5.588" extent="1-16" drill="0.508"/>
-<wire x1="15.367" y1="5.588" x2="14.008" y2="4.229" width="0.254" layer="1"/>
-<wire x1="14.008" y1="4.229" x2="9.75" y2="4.229" width="0.254" layer="1"/>
+<wire x1="15.367" y1="5.588" x2="14.726" y2="6.229" width="0.254" layer="1"/>
+<wire x1="14.726" y1="6.229" x2="9.75" y2="6.229" width="0.254" layer="1"/>
 </signal>
 <signal name="A0">
@@
 <wire x1="24.15" y1="6.878" x2="24.15" y2="7.7" width="0.2032" layer="16"/>
 </signal>
+<signal name="IN+">
+<contactref element="U100" pad="1"/>
+<contactref element="R100" pad="1"/>
+<wire x1="24.641" y1="1.524" x2="24.956" y2="2.093" width="0.508" layer="16"/>
+<wire x1="24.956" y1="2.093" x2="24.956" y2="2.8429" width="0.508" layer="16"/>
+</signal>
 </signals>
