File: NU-Smarticle PCB Design/Eagle Files/NU-Smarticles-v2.0/topboard-v2.0.sch (EAGLE design)
At the start: 17 parts, among them CON1 LI-PO, CON2 12XFFCEXTEND, M1 SERVO, M2 SERVO, U1 XBEE3, U2 INA180B2

Commit message: eagle work and files added
Parts:
- removed CON2: 12XFFCEXTEND, NU-Smarticle v2:12XFFCEXTEND
- removed R4: 10k, NU-Smarticle v2:RESISTOR_0603MP
- added CON100: 12XFFCMOLEX_51281, NU-Smarticle v2:12XFFCMOLEX_51281
- added R100: 0.1, NU-Smarticle v2:RESISTOR_0603MP
- C1: value 0.1uF -> 9.0pF
- C2: value 9.0pF -> 1.0uF
- C3: value 1.0uF -> 0.1uF
- R1: value 0.1 -> 10k
- renumbered U2 to U100
Connections:
- removed net D2: CON2.P7, U1.DOUT
- removed net D3: CON2.P8, U1.DIN
- removed net D4: CON2.P9, M1.SIG
- new net D9: CON100.P11, M1.SIG
- new net RXD1: CON100.P3, U1.DOUT
- new net TXD1: CON100.P4, U1.DIN
- net 3.3V: now also C1.2, CON100.P1, U100.VS; no longer C1.1, CON2.P10, U100.GND
- net A0: now also CON100.P6, PH2.2, R3.2; no longer CON2.P5, PH1.2, R2.2
- net A1: now also CON100.P7; no longer CON2.P4
- net A2: now also CON100.P8, PH3.2, R2.2; no longer CON2.P3, PH2.2, R3.2
- net A3: now also CON100.P9, PH1.2, R1.2; no longer CON2.P2, PH3.2, R4.2
- net D10: now also CON100.P2; no longer CON2.P0
- net GND: now also C1.1, CON100.P5, R1.1, U100.GND; no longer C1.2, CON2.P6, R4.1, U100.VS
- net N$1: now also R100.2; no longer R1.2
- net VBAT: now also CON100.P0; no longer CON2.P11
- net VCC_1: now also R100.1; no longer R1.1
Other:
- moved on the sheet: C1, C2, C3, PH1, PH2, R1, R2, R3

Commit message: delete cam outputs
Connections:
- net N$1 renamed IN-
- new net IN+: R100.1, U100.IN+
- net VCC_1: no longer R100.1, U100.IN+
Changed lines of the file:
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@@
 <net name="VCC_1" class="0">
-<segment>
-<pinref part="U100" gate="G$1" pin="IN+"/>
-<wire x1="30.48" y1="43.18" x2="30.48" y2="48.26" width="0.1524" layer="91"/>
-<pinref part="R100" gate="G$1" pin="1"/>
-<wire x1="30.48" y1="48.26" x2="30.48" y2="50.8" width="0.1524" layer="91"/>
-<junction x="30.48" y="48.26"/>
-<pinref part="SUPPLY1" gate="G$2" pin="VCC_1"/>
-</segment>
 <segment>
 <pinref part="S1" gate="1" pin="P"/>
@@
 </segment>
 </net>
-<net name="N$1" class="0">
+<net name="IN-" class="0">
 <segment>
 <pinref part="U100" gate="G$1" pin="IN-"/>
@@
 <wire x1="40.64" y1="38.1" x2="55.88" y2="38.1" width="0.1524" layer="91"/>
 <junction x="55.88" y="38.1"/>
+<label x="38.1" y="53.34" size="1.778" layer="95"/>
 </segment>
 </net>
@@
 </segment>
 </net>
+<net name="IN+" class="0">
+<segment>
+<pinref part="U100" gate="G$1" pin="IN+"/>
+<wire x1="30.48" y1="43.18" x2="30.48" y2="48.26" width="0.1524" layer="91"/>
+<pinref part="R100" gate="G$1" pin="1"/>
+<wire x1="30.48" y1="48.26" x2="30.48" y2="50.8" width="0.1524" layer="91"/>
+<junction x="30.48" y="48.26"/>
+<pinref part="SUPPLY1" gate="G$2" pin="VCC_1"/>
+<label x="27.94" y="50.8" size="1.778" layer="95"/>
+</segment>
+</net>
